File: olmBoard-hw/olmBoard-v1/olmBoard-v1.sch (KiCad schematic (older format))
At the start: 25 parts, among them J1 JST_PH, J2 Conn_A, J3 Conn_B, U1 TPS62840DLC

Commit message: Test results added
Other:
- note added: "Max Output Current: 750 mA"
Changed lines of the file:
@@
 EndData
 $EndBitmap
+Text Notes 4850 2475 0    79   Italic 16
+Max Output Current: 750 mA
 $EndSCHEMATC
